File: stm32-reflow-psu.kicad_sch (KiCad schematic)
At the start: 6 parts, among them J10 63824-1, J11 63824-1, J12 63824-1, J7 63824-1, J8 63824-1, J9 63824-1

Commit message: finalized routing and circuit schematic (so far)
Parts:
- added Q12, Q13: 2N7002, Package_TO_SOT_SMD:SOT-23, symbol Transistor_FET:2N7002
- added R4, R5: 10k, Resistor_SMD:R_0603_1608Metric, symbol Device:R_Small
- added U4: LM1117-3.3, Package_TO_SOT_SMD:SOT-223-3_TabPin2, symbol Regulator_Linear:LM1117-3.3
Connections:
- net +5V: now also J7.1, J7.2, J8.1, J8.2, U4.3 (VI)
- net GND: now also Q12.2 (S), Q13.2 (S), R4.2, R5.2, U4.1 (GND); no longer J10.1, J10.2, J9.1, J9.2
- net R1E: now also Q12.1 (G), R4.1; no longer J7.1, J7.2
- net R2E: now also Q13.1 (G), R5.1; no longer J8.1, J8.2
- new net: J9.1, J9.2, Q12.3 (D)
- new net: J10.1, J10.2, Q13.3 (D)
- new net +3V3: U4.2 (VO)
Other:
- moved on the sheet: J10, J11, J12, J8
